File: soldering_iron.kicad_sch (KiCad schematic)
At the start: 28 parts

Commit message: completed annotation
Parts:
- gave numbers to parts that had none: 28

Commit message: completed assignment of footprints
Parts:
- J3, P1: footprint (none) -> Connector:Banana_Jack_2Pin
- SW1, SW2: footprint (none) -> Button_Switch_Keyboard:SW_Cherry_MX_1.00u_PCB
Changed lines of the file:
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@@
       (effects (font (size 1.27 1.27)) (justify left))
     )
-    (property "Footprint" "" (id 2) (at 271.78 113.665 0)
+    (property "Footprint" "Connector:Banana_Jack_2Pin" (id 2) (at 271.78 113.665 0)
       (effects (font (size 1.27 1.27)) hide)
     )
@@
     (property "Reference" "SW2" (id 0) (at 198.12 106.68 0))
     (property "Value" "SW_Push" (id 1) (at 198.12 109.22 0))
-    (property "Footprint" "" (id 2) (at 198.12 109.22 0)
+    (property "Footprint" "Button_Switch_Keyboard:SW_Cherry_MX_1.00u_PCB" (id 2) (at 198.12 109.22 0)
       (effects (font (size 1.27 1.27)) hide)
     )
@@
     (property "Reference" "P1" (id 0) (at 140.335 146.05 0))
     (property "Value" "Plug" (id 1) (at 140.97 147.955 0))
-    (property "Footprint" "" (id 2) (at 136.525 147.32 0)
+    (property "Footprint" "Connector:Banana_Jack_2Pin" (id 2) (at 136.525 147.32 0)
       (effects (font (size 1.27 1.27)) hide)
     )
@@
     (property "Reference" "SW1" (id 0) (at 197.485 120.65 0))
     (property "Value" "SW_Push" (id 1) (at 197.485 123.19 0))
-    (property "Footprint" "" (id 2) (at 197.485 123.19 0)
+    (property "Footprint" "Button_Switch_Keyboard:SW_Cherry_MX_1.00u_PCB" (id 2) (at 197.485 123.19 0)
       (effects (font (size 1.27 1.27)) hide)
     )
@@
     )
     (path "/209f41bc-f707-4dab-a5ba-398a64e1e109"
-      (reference "J3") (unit 1) (value "VIBRATOR") (footprint "")
+      (reference "J3") (unit 1) (value "VIBRATOR") (footprint "Connector:Banana_Jack_2Pin")
     )
     (path "/b7d633b1-9984-4680-89c4-ee6032cb59ba"
-      (reference "P1") (unit 1) (value "Plug") (footprint "")
+      (reference "P1") (unit 1) (value "Plug") (footprint "Connector:Banana_Jack_2Pin")
     )
     (path "/ba3bb3ff-9a2f-4de5-ba97-3a9491ea9505"
@@
     )
     (path "/f78108b4-edef-4259-81ef-b242f7e55a74"
-      (reference "SW1") (unit 1) (value "SW_Push") (footprint "")
+      (reference "SW1") (unit 1) (value "SW_Push") (footprint "Button_Switch_Keyboard:SW_Cherry_MX_1.00u_PCB")
     )
     (path "/5207b551-fedd-4955-9c18-eea2162cea82"
-      (reference "SW2") (unit 1) (value "SW_Push") (footprint "")
+      (reference "SW2") (unit 1) (value "SW_Push") (footprint "Button_Switch_Keyboard:SW_Cherry_MX_1.00u_PCB")
     )
     (path "/658cbe5a-e7f5-4f80-bc14-54c2ecfeca7c"
